File: The Supluwu PCB/5V Regulator.kicad_sch (KiCad schematic)
At the start: 15 parts, among them IC2 RT6285GSP

Commit message: added 3D
Other:
- note added: "PM4343.15NLT"
Changed lines of the file:
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@@
+    (effects (font (size 1.27 1.27)) (justify left bottom))
+  )
+  (text "PM4343.15NLT" (at 171.45 79.375 0)
     (effects (font (size 1.27 1.27)) (justify left bottom))
   )
